Commit message: fixed IrisInConfigurationSpace error

File: data/unload-gen0/robot_base.urdf (robot description, URDF)
Before this commit: robot unload-gen0, 16 links, 15 joints
Joints:
- joint base_footprint_frame: limit (none) -> lower=0.0 upper=0.0
- joint base_front_left_frame: limit (none) -> lower=0.0 upper=0.0
- joint base_link_to_base: limit (none) -> lower=0.0 upper=0.0
- joint base_rear_left_frame: limit (none) -> lower=0.0 upper=0.0
- joint base_top_frame: limit (none) -> lower=0.0 upper=0.0
- joint base_top_left_frame: limit (none) -> lower=0.0 upper=0.0
- joint base_top_right_frame: limit (none) -> lower=0.0 upper=0.0
- joint caster_center_frame: limit (none) -> lower=0.0 upper=0.0
- joint conveyor_front_right_frame: limit (none) -> lower=0.0 upper=0.0
- joint conveyor_rear_right_frame: limit (none) -> lower=0.0 upper=0.0
- joint mobile_base_frame: limit (none) -> lower=0.0 upper=0.0
- joint wheel_width_left_frame: limit (none) -> lower=0.0 upper=0.0
- joint wheel_width_right_frame: limit (none) -> lower=0.0 upper=0.0

Commit message: robot_base converted to box primitives for collision geometries

File: data/unload-gen0/robot_base.urdf (robot description, URDF)
Before this commit: robot unload-gen0, 16 links, 15 joints
Links:
- link base: geometry collision box size=2.4173 0.99 0.246; visual mesh filename=base_detailed.obj
- link base_top_left: geometry collision box size=0.9657 0.18 0.35757
- link base_top_right: geometry collision box size=1.1257 0.18 0.35757
- link conveyor_front_right: geometry collision box size=2.6 0.6336 0.5164
- link right_motor: geometry visual mesh filename=wheel.obj
