Commit message: removed sensor tower from collision geometry; not possible for the arm to hit it anyway + causing fake collisions

File: data/unload-gen0/robot_arm.urdf (robot description, URDF)
Before this commit: robot kuka, 10 links, 9 joints
Links:
- link arm_a1: geometry collision mesh filename=krl70_a1_part_10.obj; collision mesh filename=krl70_a1_part_13.obj

File: data/unload-gen0/robot_base.urdf (robot description, URDF)
Before this commit: robot unload-gen0, 14 links, 13 joints
Links:
- added link base_top_left, mass 1e-9; collision mesh filename=Base_split_top_left.obj
- added link base_top_right, mass 1e-9; collision mesh filename=Base_split_top_right.obj
- link base_top: geometry collision mesh filename=Base_split_top_mid.obj
Joints:
- added joint base_top_left_frame: type fixed, parent base, child base_top_left, origin xyz=-3.4254225040659449532e-17 0 1.6163685799999993886 rpy=0 -0 0, axis 0 0 0
- added joint base_top_right_frame: type fixed, parent base, child base_top_right, origin xyz=-3.4254225040659449532e-17 0 1.6163685799999993886 rpy=0 -0 0, axis 0 0 0

Commit message: fixed creation of MBP in gcs.py so that it now takes into account collisions

File: data/unload-gen0/robot_arm.urdf (robot description, URDF)
Before this commit: robot kuka, 10 links, 9 joints
Links:
- link arm_a6: geometry collision mesh filename=krl70_a5_part_2.obj; collision mesh filename=krl70_a6_part_1.obj

Commit message: debugging leafsytem

File: data/unload-gen0/robot_arm.urdf (robot description, URDF)
Before this commit: robot kuka, 10 links, 9 joints
Joints:
- joint arm_a1: limit lower=-3.05432619099 upper=3.05432619099 effort=1 velocity=20 -> lower=-2.09439510239 upper=2.09439510239 effort=10000 velocity=1.4835298641951802
- joint arm_a2: limit lower=-3.05432619099 upper=3.05432619099 effort=1 velocity=20 -> lower=-2.09439510239 upper=2.09439510239 effort=10000 velocity=1.4835298641951802
- joint arm_a3: limit lower=-3.05432619099 upper=3.05432619099 effort=1 velocity=20 -> lower=-2.09439510239 upper=2.09439510239 effort=10000 velocity=1.4835298641951802
- joint arm_a4: limit lower=-3.05432619099 upper=3.05432619099 effort=1 velocity=20 -> lower=-2.09439510239 upper=2.09439510239 effort=10000 velocity=1.4835298641951802
- joint arm_a5: limit lower=-3.05432619099 upper=3.05432619099 effort=1 velocity=20 -> lower=-2.09439510239 upper=2.09439510239 effort=10000 velocity=1.4835298641951802
- joint arm_a6: limit lower=-3.05432619099 upper=3.05432619099 effort=1 velocity=20 -> lower=-2.09439510239 upper=2.09439510239 effort=10000 velocity=1.4835298641951802

Commit message: debuggig

File: data/unload-gen0/robot_arm.urdf (robot description, URDF)
Before this commit: robot kuka, 10 links, 9 joints
Joints:
- joint arm_a1: limit lower=-2.09439510239 upper=2.09439510239 effort=10000 velocity=1.4835298641951802 -> lower=-3.22886 upper=3.22886 effort=10000 velocity=1.4835298641951802
- joint arm_a2: limit lower=-2.09439510239 upper=2.09439510239 effort=10000 velocity=1.4835298641951802 -> lower=-3.05433 upper=1.0472 effort=10000 velocity=1.4835298641951802
- joint arm_a3: limit lower=-2.09439510239 upper=2.09439510239 effort=10000 velocity=1.4835298641951802 -> lower=-2.09439510239 upper=2.87979 effort=10000 velocity=1.4835298641951802
- joint arm_a4: limit lower=-2.09439510239 upper=2.09439510239 effort=10000 velocity=1.4835298641951802 -> lower=-3.141592 upper=3.141592 effort=10000 velocity=1.4835298641951802
- joint arm_a5: limit lower=-2.09439510239 upper=2.09439510239 effort=10000 velocity=1.4835298641951802 -> lower=-2.18166 upper=2.18166 effort=10000 velocity=1.4835298641951802
- joint arm_a6: limit lower=-2.09439510239 upper=2.09439510239 effort=10000 velocity=1.4835298641951802 -> lower=-6.10865 upper=6.10865 effort=10000 velocity=1.4835298641951802

Commit message: fixed inversedynamics bug--needed to reorder transmission tags in urdf

File: data/unload-gen0/robot_arm.urdf (robot description, URDF)
Before this commit: robot kuka, 10 links, 9 joints
Links:
- removed link camera_mast_top
- link arm_a1: geometry collision mesh filename=krl70_a1_surface_1.obj; visual mesh filename=krl70_a1_surface_1.obj
- link arm_a3: geometry collision mesh filename=krl70_a3_part_1.obj; visual mesh filename=krl70_a3_part_1.obj
- link arm_a6: mass 20 -> 10; geometry collision mesh filename=krl70_a6_part_1.obj; visual mesh filename=krl70_a6_part_1.obj
Joints:
- removed joint camera_mast_top_frame

Commit message: cleaned up from debugging

File: data/unload-gen0/robot_arm.urdf (robot description, URDF)
Before this commit: robot kuka, 9 links, 8 joints
Links:
- link arm_a1: geometry collision mesh filename=krl70_a1_part_10.obj; collision mesh filename=krl70_a1_part_13.obj
- link arm_a3: geometry collision mesh filename=krl70_a3_part_1.obj; collision mesh filename=krl70_a3_part_4.obj
- link arm_a6: geometry collision mesh filename=krl70_a5_part_2.obj; collision mesh filename=krl70_a6_part_1.obj

Commit message: attempted visualization of cspace

File: data/unload-gen0/robot_arm.urdf (robot description, URDF)
Before this commit: robot kuka, 9 links, 8 joints
Joints:
- joint arm_a1: limit lower=-3.22886 upper=3.22886 effort=10000 velocity=1.4835298641951802 -> lower=-3.15 upper=3.15 effort=10000 velocity=1.4835298641951802
- joint arm_a6: limit lower=-6.10865 upper=6.10865 effort=10000 velocity=1.4835298641951802 -> lower=-3.15 upper=3.15 effort=10000 velocity=1.4835298641951802

Commit message: box collision geometries on robot arm, experiment results, iris region testing improvements

File: data/unload-gen0/robot_arm.urdf (robot description, URDF)
Before this commit: robot kuka, 9 links, 8 joints
Links:
- link arm_a1: geometry collision box size=0.65 0.6 0.6; visual mesh filename=krl70_a1_part_10.obj
- link arm_a2: geometry collision box size=1.1 0.21 0.16; visual mesh filename=krl70_a2_surface_1.obj
- link arm_a3: geometry collision box size=0.4 0.24 0.705; visual mesh filename=krl70_a3_part_1.obj
- link arm_a4: geometry collision box size=0.15 0.2 0.91; visual mesh filename=krl70_a4_part_1.obj
- link arm_a5: geometry collision box size=0.16 0.27 0.185; visual mesh filename=krl70_a5_part_1.obj
- link arm_a6: geometry collision box size=0.25 0.25 0.05; visual mesh filename=krl70_a5_part_2.obj
- link arm_base: geometry collision box size=0.46 0.46 0.2; visual mesh filename=krl70_a0_surface_1.obj
Joints:
- joint arm_a1: origin xyz=6.9388939039072276073e-18 1.0408340855860842566e-17 0.16999995708465576172 rpy=-3.141592653589793116 1.7783981468004833182e-49 1.570796326794896336 -> xyz=6.9388939039072276073e-18 1.0408340855860842566e-17 0.16999995708465576172 rpy=-3.141592653589793116 0 1.570796326794896336
- joint arm_a2: origin xyz=-0.10723578937805347544 0.17450280203385484801 -0.40497676867967002945 rpy=1.570796326794896558 -2.2204460492503431562e-16 1.570796326794896558 -> xyz=-0.10723578937805347544 0.17450280203385484801 -0.40497676867967002945 rpy=1.570796326794896558 0 1.570796326794896558

File: data/unload-gen0/robot_base.urdf (robot description, URDF)
Before this commit: robot unload-gen0, 16 links, 15 joints
Links:
- link base_front_left: geometry 
- link base_rear_left: geometry 
- link base_top: geometry 
- link caster_center: geometry 
- link left_motor: geometry visual mesh filename=wheel.obj
- link mobile_base: geometry 

Commit message: pipeline running except 1 ik failure??

File: data/unload-gen0/robot_arm.urdf (robot description, URDF)
Before this commit: robot kuka, 9 links, 8 joints
Links:
- link arm_a1: geometry collision box size=0.55 0.5 0.6; visual mesh filename=krl70_a1_part_10.obj

Commit message: bug fixes and corrected joint limits

File: data/unload-gen0/robot_arm.urdf (robot description, URDF)
Before this commit: robot kuka, 9 links, 8 joints
Joints:
- joint arm_a3: limit lower=-2.09439510239 upper=2.87979 effort=10000 velocity=1.4835298641951802 -> lower=-0.33 upper=2.87979 effort=10000 velocity=1.4835298641951802
- joint arm_a6: limit lower=-3.15 upper=3.15 effort=10000 velocity=1.4835298641951802 -> lower=-3.141592 upper=3.141592 effort=10000 velocity=1.4835298641951802
